File: VoltV1/daughterInterface.kicad_sch (KiCad schematic)
At the start: 1 part, among them J2 SFM-120-02-X-D-A

Commit message: merging. power stuff incomplete
Connections:
- net Daughter Battery: now reaches J2.01
- net Daughter Battery: now also J2.03, J2.05
- net Daughter 5V: now reaches J2.02
- net Daughter 5V: now also J2.04
- net Daughter 3.3V: now reaches J2.06
Changed lines of the file:
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@@
+		)
+	)
+	(hierarchical_label "Daughter 5V"
+		(shape input)
+		(at 158.75 74.93 0)
+		(effects
+			(font
+				(size 1.27 1.27)
+			)
+			(justify left)
 		)
 	)
@@
 		)
 	)
+	(hierarchical_label "Daughter 5V"
+		(shape input)
+		(at 158.75 77.47 0)
+		(effects
+			(font
+				(size 1.27 1.27)
+			)
+			(justify left)
+		)
+	)
 	(hierarchical_label "DaughterPWM{slash}Analogue3"
 		(shape input)
@@
 		)
 	)
+	(hierarchical_label "Daughter Battery"
+		(shape input)
+		(at 133.35 80.01 180)
+		(effects
+			(font
+				(size 1.27 1.27)
+			)
+			(justify right)
+		)
+	)
 	(hierarchical_label "~S4.3"
 		(shape input)
@@
 		)
 	)
+	(hierarchical_label "Daughter Battery"
+		(shape input)
+		(at 133.35 77.47 180)
+		(effects
+			(font
+				(size 1.27 1.27)
+			)
+			(justify right)
+		)
+	)
 	(hierarchical_label "DAC0"
 		(shape input)
@@
 		)
 	)
+	(hierarchical_label "Daughter Battery"
+		(shape input)
+		(at 133.35 74.93 180)
+		(effects
+			(font
+				(size 1.27 1.27)
+			)
+			(justify right)
+		)
+	)
 	(hierarchical_label "DaughterPWM{slash}Analogue1"
 		(shape input)
@@
 		)
 	)
+	(hierarchical_label "Daughter 3.3V"
+		(shape input)
+		(at 158.75 80.01 0)
+		(effects
+			(font
+				(size 1.27 1.27)
+			)
+			(justify left)
+		)
+	)
