File: VoltV1/VoltV1.kicad_sch (KiCad schematic)
At the start: 0 parts

Commit message: merging. power stuff incomplete
Other:
- sheet daughterInterface ports: added Daughter 3.3V, Daughter 5V, Daughter Battery; removed none
- sheet mcu ports: added ICM Int1, ICM20948 CS; removed none
- sheet power ports: added Daughter 3.3V, Daughter 5V, USBD+, USBD-; removed none
- sheet sensors ports: added ICM Int1, ICM20948 CS; removed none
- company: (none) -> Riley Post
Changed lines of the file:
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@@
 	(title_block
 		(title "Volt")
+		(date "2026-03-05")
 		(rev "V1")
+		(company "Riley Post")
 	)
 	(text "NULI-Avionics PCBs"
@@
 	(wire
 		(pts
+			(xy 71.12 46.99) (xy 64.77 46.99)
+		)
+		(stroke
+			(width 0)
+			(type default)
+		)
+	)
+	(wire
+		(pts
 			(xy 109.22 162.56) (xy 127 162.56)
 		)
@@
 	(wire
 		(pts
+			(xy 62.23 44.45) (xy 62.23 67.31)
+		)
+		(stroke
+			(width 0)
+			(type default)
+		)
+	)
+	(wire
+		(pts
 			(xy 193.04 99.06) (xy 208.28 99.06)
 		)
@@
 	(wire
 		(pts
+			(xy 109.22 27.94) (xy 127 27.94)
+		)
+		(stroke
+			(width 0)
+			(type default)
+		)
+	)
+	(wire
+		(pts
 			(xy 172.72 153.67) (xy 207.01 153.67)
 		)
@@
 	(wire
 		(pts
+			(xy 71.12 44.45) (xy 62.23 44.45)
+		)
+		(stroke
+			(width 0)
+			(type default)
+		)
+	)
+	(wire
+		(pts
 			(xy 172.72 64.77) (xy 208.28 64.77)
 		)
@@
 	(wire
 		(pts
+			(xy 109.22 30.48) (xy 127 30.48)
+		)
+		(stroke
+			(width 0)
+			(type default)
+		)
+	)
+	(wire
+		(pts
 			(xy 107.95 77.47) (xy 127 77.47)
 		)
@@
 	(wire
 		(pts
+			(xy 172.72 128.27) (xy 207.01 128.27)
+		)
+		(stroke
+			(width 0)
+			(type default)
+		)
+	)
+	(wire
+		(pts
 			(xy 172.72 143.51) (xy 207.01 143.51)
 		)
@@
 	(wire
 		(pts
+			(xy 64.77 64.77) (xy 69.85 64.77)
+		)
+		(stroke
+			(width 0)
+			(type default)
+		)
+	)
+	(wire
+		(pts
 			(xy 172.72 138.43) (xy 207.01 138.43)
 		)
@@
 	(wire
 		(pts
+			(xy 172.72 130.81) (xy 207.01 130.81)
+		)
+		(stroke
+			(width 0)
+			(type default)
+		)
+	)
+	(wire
+		(pts
 			(xy 172.72 31.75) (xy 208.28 31.75)
 		)
@@
 		)
 	)
+	(wire
+		(pts
+			(xy 64.77 46.99) (xy 64.77 64.77)
+		)
+		(stroke
+			(width 0)
+			(type default)
+		)
+	)
+	(wire
+		(pts
+			(xy 62.23 67.31) (xy 69.85 67.31)
+		)
+		(stroke
+			(width 0)
+			(type default)
+		)
+	)
 	(sheet
-		(at 207.01 115.57)
-		(size 38.1 45.72)
+		(at 207.01 124.46)
+		(size 38.1 36.83)
 		(exclude_from_sim no)
 		(in_bom yes)
@@
 		)
 		(property "Sheetname" "sensors"
-			(at 207.01 114.8584 0)
+			(at 207.01 123.7484 0)
 			(effects
 				(font
@@
 		(pin "Sck1" input
 			(at 207.01 156.21 180)
+			(effects
+				(font
+					(size 1.27 1.27)
+				)
+				(justify left)
+			)
+		)
+		(pin "ICM20948 CS" input
+			(at 207.01 130.81 180)
+			(effects
+				(font
+					(size 1.27 1.27)
+				)
+				(justify left)
+			)
+		)
+		(pin "ICM Int1" input
+			(at 207.01 128.27 180)
 			(effects
 				(font
@@
 			)
 		)
+		(pin "Daughter 3.3V" input
+			(at 71.12 46.99 180)
+			(effects
+				(font
+					(size 1.27 1.27)
+				)
+				(justify left)
+			)
+		)
+		(pin "Daughter 5V" input
+			(at 71.12 44.45 180)
+			(effects
+				(font
+					(size 1.27 1.27)
+				)
+				(justify left)
+			)
+		)
+		(pin "USBD+" input
+			(at 109.22 27.94 0)
+			(effects
+				(font
+					(size 1.27 1.27)
+				)
+				(justify right)
+			)
+		)
+		(pin "USBD-" input
+			(at 109.22 30.48 0)
+			(effects
+				(font
+					(size 1.27 1.27)
+				)
+				(justify right)
+			)
+		)
 		(instances
 			(project "VoltV1"
@@
 		)
 		(pin "GPIOspare0" input
-			(at 127 41.91 180)
+			(at 127 95.25 180)
 			(effects
 				(font
@@
 		)
 		(pin "GPIOspare1" input
-			(at 127 39.37 180)
+			(at 127 97.79 180)
 			(effects
 				(font
@@
 		)
 		(pin "GPIOspare2" input
-			(at 127 36.83 180)
+			(at 127 100.33 180)
 			(effects
 				(font
@@
 				)
 				(justify left)
+			)
+		)
+		(pin "ICM20948 CS" input
+			(at 172.72 130.81 0)
+			(effects
+				(font
+					(size 1.27 1.27)
+				)
+				(justify right)
+			)
+		)
+		(pin "ICM Int1" input
+			(at 172.72 128.27 0)
+			(effects
+				(font
+					(size 1.27 1.27)
+				)
+				(justify right)
 			)
 		)
@@
 			)
 		)
+		(pin "Daughter 3.3V" input
+			(at 69.85 64.77 180)
+			(effects
+				(font
+					(size 1.27 1.27)
+				)
+				(justify left)
+			)
+		)
+		(pin "Daughter 5V" input
+			(at 69.85 67.31 180)
+			(effects
+				(font
+					(size 1.27 1.27)
+				)
+				(justify left)
+			)
+		)
+		(pin "Daughter Battery" input
+			(at 69.85 69.85 180)
+			(effects
+				(font
+					(size 1.27 1.27)
+				)
+				(justify left)
+			)
+		)

Commit message: updates to schematic
Parts:
- added H1, H2, H3, H4: MountingHole, M25Fixed:FixedMountingHole_2.5mm_Pad, symbol Mechanical:MountingHole
Other:
- sheet GPSRadio ports: added none; removed RxEn Radio, TxEN Radio
- sheet IO ports: added RESETN, SWCLK, SWDIO; removed none
- sheet power ports: added CurrentDetection, Daughter Batt+; removed none
