File: VoltV1/GPSRadio.kicad_sch (KiCad schematic)
At the start: 12 parts, among them J3 Conn_Coaxial, J4 Conn_Coaxial, U3 MAX-M10S-00B, U9 E22-900M30S

Commit message: merging. power stuff incomplete
Parts:
- added R26: 100k, Resistor_SMD:R_0603_1608Metric, symbol Device:R_Small
Connections:
- net +3V3: now also R26.2
- net CS Radio: now also R26.1
Changed lines of the file:
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@@
+	)
+	(junction
+		(at 170.18 83.82)
+		(diameter 0)
+		(color 0 0 0 0)
 	)
 	(junction
@@
 	(wire
 		(pts
+			(xy 170.18 63.5) (xy 170.18 73.66)
+		)
+		(stroke
+			(width 0)
+			(type default)
+		)
+	)
+	(wire
+		(pts
 			(xy 248.92 83.82) (xy 248.92 86.36)
 		)
@@
 	(wire
 		(pts
+			(xy 170.18 78.74) (xy 170.18 83.82)
+		)
+		(stroke
+			(width 0)
+			(type default)
+		)
+	)
+	(wire
+		(pts
 			(xy 119.38 68.58) (xy 119.38 66.04)
 		)
@@
 	(wire
 		(pts
+			(xy 163.83 83.82) (xy 170.18 83.82)
+		)
+		(stroke
+			(width 0)
+			(type default)
+		)
+	)
+	(wire
+		(pts
 			(xy 222.25 96.52) (xy 222.25 99.06)
 		)
@@
 		(pts
 			(xy 124.46 66.04) (xy 129.54 66.04)
+		)
+		(stroke
+			(width 0)
+			(type default)
+		)
+	)
+	(wire
+		(pts
+			(xy 170.18 83.82) (xy 186.69 83.82)
 		)
 		(stroke
@@
 	(hierarchical_label "CS Radio"
 		(shape input)
-		(at 186.69 83.82 180)
+		(at 163.83 83.82 180)
 		(effects
 			(font
@@
 	)
 	(symbol
+		(lib_id "power:+3.3V")
+		(at 170.18 63.5 0)
+		(unit 1)
+		(exclude_from_sim no)
+		(in_bom yes)
+		(on_board yes)
+		(dnp no)
+		(property "Reference" "#PWR025"
+			(at 170.18 67.31 0)
+			(effects
+				(font
+					(size 1.27 1.27)
+				)
+				(hide yes)
+			)
+		)
+		(property "Value" "+3V3"
+			(at 170.5483 59.1756 0)
+			(effects
+				(font
+					(size 1.27 1.27)
+				)
+			)
+		)
+		(property "Footprint" ""
+			(at 170.18 63.5 0)
+			(effects
+				(font
+					(size 1.27 1.27)
+				)
+			)
+		)
+		(property "Datasheet" ""
+			(at 170.18 63.5 0)
+			(effects
+				(font
+					(size 1.27 1.27)
+				)
+			)
+		)
+		(property "Description" "Power symbol creates a global label with name \"+3.3V\""
+			(at 170.18 63.5 0)
+			(effects
+				(font
+					(size 1.27 1.27)
+				)
+				(hide yes)
+			)
+		)
+		(pin "1"
+		)
+		(instances
+			(project "VoltV1"
+				(path "/4dc02877-6404-4472-a9f6-00d826e215ba/c4a60ef4-4a9e-46a3-8362-ab2012feb48c"
+					(reference "#PWR025")
+					(unit 1)
+				)
+			)
+		)
+	)
+	(symbol
 		(lib_id "Device:R_Small")
 		(at 48.26 71.12 270)
@@
 					(unit 1)
 				)
+			)
+		)
+	)
+	(symbol
+		(lib_id "Device:R_Small")
+		(at 170.18 76.2 180)
+		(unit 1)
+		(exclude_from_sim no)
+		(in_bom yes)
+		(on_board yes)
+		(dnp no)
+		(property "Reference" "R26"
+			(at 167.64 73.66 90)
+			(effects
+				(font
+					(size 1.27 1.27)
+				)
+			)
+		)
+		(property "Value" "100k"
+			(at 165.1 73.66 90)
+			(effects
+				(font
+					(size 1.27 1.27)
+				)
+			)
+		)
+		(property "Footprint" "Resistor_SMD:R_0603_1608Metric"
+			(at 170.18 76.2 0)
+			(effects
+				(font
+					(size 1.27 1.27)
+				)
+				(hide yes)
+			)
+		)
+		(property "Datasheet" "~"
+			(at 170.18 76.2 0)
+			(effects
+				(font
+					(size 1.27 1.27)
+				)
+				(hide yes)
+			)
+		)
+		(property "Description" ""
+			(at 170.18 76.2 0)
+			(effects
+				(font
+					(size 1.27 1.27)
+				)
+			)
+		)
+		(property "LCSC" "C25077"
+			(at 170.18 76.2 90)
+			(effects
+				(font
+					(size 1.27 1.27)
+				)
+				(hide yes)
+			)
+		)
+		(pin "1"
+		)
+		(pin "2"
+		)
+		(instances
+			(project "VoltV1"
+				(path "/4dc02877-6404-4472-a9f6-00d826e215ba/c4a60ef4-4a9e-46a3-8362-ab2012feb48c"
+					(reference "R26")
+					(unit 1)
+				)

Commit message: updates to schematic
Parts:
- removed C27, C28: .1uF, Capacitor_SMD:C_0603_1608Metric, symbol Device:C
- removed C29: 10uF, Capacitor_SMD:C_0603_1608Metric, symbol Device:C
- removed C32: 10nF, Capacitor_SMD:C_0603_1608Metric, symbol Device:C_Small
- removed J3, J4: Conn_Coaxial, Connector_Coaxial:SMA_Molex_73251-1153_EdgeMount_Horizontal, symbol Connector:Conn_Coaxial
- removed L3: 27n, Inductor_SMD:L_0603_1608Metric, symbol Device:L_Small
- removed R8: 10, Resistor_SMD:R_0603_1608Metric, symbol Device:R_Small
- removed U3: MAX-M10S-00B, VOLTV1:XCVR_MAX-M10S-00B, symbol VOLTV1:MAX-M10S-00B
- removed U9: E22-900M30S, VOLTV1:XCVR_E22-900M30S, symbol VOLTV1:E22-900M30S
- added D8: LED, LED_SMD:LED_0603_1608Metric, symbol Device:LED
- added R8: 270, Resistor_SMD:R_0603_1608Metric, symbol Device:R
- added U15: SAM-M8Q, RF_GPS:ublox_SAM-M8Q, symbol RF_GPS:SAM-M8Q
Connections:
- net +3V3: now also U15.17 (VCC), U15.2 (VCC_IO), U15.3 (V_BCKP)
- net GND: now also D8.1 (K), U15.1 (GND), U15.10 (GND), U15.11 (GND), U15.15 (GND), U15.16 (GND), U15.20 (GND), U15.4 (GND), U15.5 (GND), U15.6 (GND)
- net RxGPS: now also U15.14 (RXD)
- net TxGPS: now also U15.13 (TXD)
- new net: R8.1, U15.7 (TIMEPULSE)
- new net: D8.2 (A), R8.2
- no-connect marks 7 -> 4
Other:
- added sheet Radio (radio.kicad_sch)
- note added: "Do we want a backup battery?"
- note removed: "50 Ohm Impedance"
- moved on the sheet: C30, C31, R26

Commit message: schematic updates
Parts:
- C30, C31: footprint Capacitor_SMD:C_0603_1608Metric -> Capacitor_SMD:C_0402_1005Metric
- R26, R8: footprint Resistor_SMD:R_0603_1608Metric -> Resistor_SMD:R_0402_1005Metric
Changed lines of the file:
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@@
 			)
 		)
-		(property "Footprint" "Resistor_SMD:R_0603_1608Metric"
+		(property "Footprint" "Resistor_SMD:R_0402_1005Metric"
 			(at 42.672 152.4 90)
 			(effects
@@
 			)
 		)
-		(property "Footprint" "Capacitor_SMD:C_0603_1608Metric"
+		(property "Footprint" "Capacitor_SMD:C_0402_1005Metric"
 			(at 85.3948 111.76 0)
 			(effects
@@
 			)
 		)
-		(property "Footprint" "Capacitor_SMD:C_0603_1608Metric"
+		(property "Footprint" "Capacitor_SMD:C_0402_1005Metric"
 			(at 80.3148 111.76 0)
 			(effects
@@
 			)
 		)
-		(property "Footprint" "Resistor_SMD:R_0603_1608Metric"
+		(property "Footprint" "Resistor_SMD:R_0402_1005Metric"
 			(at 190.5 71.12 0)
 			(effects
