File: VoltV1/IO.kicad_sch (KiCad schematic)
At the start: 8 parts, among them Q4 IRLML6244

Commit message: merging. power stuff incomplete
Other:
- moved on the sheet: D1, R18
Changed lines of the file:
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@@
 	(text "(3.3-2.85)/(2mA/1000)\n=225 ohnm min"
 		(exclude_from_sim no)
-		(at 59.436 88.9 0)
+		(at 70.866 88.9 0)
 		(effects
 			(font
@@
 	(wire
 		(pts
-			(xy 76.2 85.09) (xy 76.2 82.55)
+			(xy 87.63 85.09) (xy 87.63 82.55)
 		)
 		(stroke
@@
 	(wire
 		(pts
-			(xy 76.2 102.87) (xy 76.2 101.6)
+			(xy 87.63 102.87) (xy 87.63 101.6)
 		)
 		(stroke
@@
 	(wire
 		(pts
-			(xy 76.2 92.71) (xy 76.2 93.98)
+			(xy 87.63 92.71) (xy 87.63 93.98)
 		)
 		(stroke
@@
 	(hierarchical_label "LEDio"
 		(shape input)
-		(at 76.2 82.55 90)
+		(at 87.63 82.55 90)
 		(effects
 			(font
@@
 	(symbol
 		(lib_id "Device:R")
-		(at 76.2 88.9 0)
+		(at 87.63 88.9 0)
 		(unit 1)
 		(exclude_from_sim no)
@@
 		(dnp no)
 		(property "Reference" "R18"
-			(at 77.47 87.63 0)
+			(at 88.9 87.63 0)
 			(effects
 				(font
@@
 		)
 		(property "Value" "270"
-			(at 78.74 91.44 0)
+			(at 90.17 91.44 0)
 			(effects
 				(font
@@
 		)
 		(property "Footprint" "Resistor_SMD:R_0603_1608Metric"
-			(at 74.422 88.9 90)
+			(at 85.852 88.9 90)
 			(effects
 				(font
@@
 		)
 		(property "Datasheet" "~"
-			(at 76.2 88.9 0)
+			(at 87.63 88.9 0)
 			(effects
 				(font
@@
 		)
 		(property "Description" "Resistor"
-			(at 76.2 88.9 0)
+			(at 87.63 88.9 0)
 			(effects
 				(font
@@
 	(symbol
 		(lib_id "Device:LED")
-		(at 76.2 97.79 90)
+		(at 87.63 97.79 90)
 		(unit 1)
 		(exclude_from_sim no)
@@
 		(fields_autoplaced yes)
 		(property "Reference" "D1"
-			(at 69.85 99.3775 0)
+			(at 81.28 99.3775 0)
 			(effects
 				(font
@@
 		)
 		(property "Value" "LED"
-			(at 72.39 99.3775 0)
+			(at 83.82 99.3775 0)
 			(effects
 				(font
@@
 		)
 		(property "Footprint" "LED_SMD:LED_0603_1608Metric"
-			(at 76.2 97.79 0)
+			(at 87.63 97.79 0)
 			(effects
 				(font
@@
 		)
 		(property "Datasheet" "~"
-			(at 76.2 97.79 0)
+			(at 87.63 97.79 0)
 			(effects
 				(font
@@
 		)
 		(property "Description" "Light emitting diode"
-			(at 76.2 97.79 0)
+			(at 87.63 97.79 0)
 			(effects
 				(font
@@
 	(symbol
 		(lib_id "power:GND")
-		(at 76.2 102.87 0)
+		(at 87.63 102.87 0)
 		(unit 1)
 		(exclude_from_sim no)
@@
 		(fields_autoplaced yes)
 		(property "Reference" "#PWR042"
-			(at 76.2 109.22 0)
+			(at 87.63 109.22 0)
 			(effects
 				(font
@@
 		)
 		(property "Value" "GND"
-			(at 76.1999 106.68 90)
+			(at 87.6299 106.68 90)
 			(effects
 				(font
@@
 		)
 		(property "Footprint" ""
-			(at 76.2 102.87 0)
+			(at 87.63 102.87 0)
 			(effects
 				(font
@@
 		)
 		(property "Datasheet" ""
-			(at 76.2 102.87 0)
+			(at 87.63 102.87 0)
 			(effects
 				(font
@@
 		)
 		(property "Description" "Power symbol creates a global label with name \"GND\" , ground"
-			(at 76.2 102.87 0)
-			(effects
-				(font
+			(at 87.63 102.87 0)
+			(effects
+				(font

Commit message: updates to schematic
Parts:
- removed LS1: CMT-0525-75-SMT-TR, CMT-0525-75-SMT-TR:XDCR_CMT-0525-75-SMT-TR, symbol CMT-0525-75-SMT-TR:CMT-0525-75-SMT-TR
- added J7: Conn_01x08, Connector_JST:JST_GH_BM08B-GHS-TBT_1x08-1MP_P1.25mm_Vertical, symbol Connector_Generic:Conn_01x08
- added LS1: CMT-0525-75-SMT-TR, VOLTV1:XDCR_CMT-0525-75-SMT-TR, symbol VOLTV1:CMT-0525-75-SMT-TR
Connections:
- net +3.3V: now also J7.2 (Pin_2)
- net GND: now also J7.1 (Pin_1)
- net at D3.2 (A), Q4.3 (D): now also LS1.N
- net at D3.1 (K), R25.2: now also LS1.P
- new net RESETN: J7.5 (Pin_5)
- new net SWCLK: J7.4 (Pin_4)
- new net SWDIO: J7.3 (Pin_3)

Commit message: schematic updates
Parts:
- R18, R23, R24, R25: footprint Resistor_SMD:R_0603_1608Metric -> Resistor_SMD:R_0402_1005Metric
Changed lines of the file:
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@@
 			)
 		)
-		(property "Footprint" "Resistor_SMD:R_0603_1608Metric"
+		(property "Footprint" "Resistor_SMD:R_0402_1005Metric"
 			(at 140.97 104.648 90)
 			(effects
@@
 			)
 		)
-		(property "Footprint" "Resistor_SMD:R_0603_1608Metric"
+		(property "Footprint" "Resistor_SMD:R_0402_1005Metric"
 			(at 85.852 88.9 90)
 			(effects
@@
 			)
 		)
-		(property "Footprint" "Resistor_SMD:R_0603_1608Metric"
+		(property "Footprint" "Resistor_SMD:R_0402_1005Metric"
 			(at 155.702 71.12 90)
 			(effects
@@
 			)
 		)
-		(property "Footprint" "Resistor_SMD:R_0603_1608Metric"
+		(property "Footprint" "Resistor_SMD:R_0402_1005Metric"
 			(at 149.098 107.95 90)
 			(effects
