File: VoltV1/Pyros.kicad_sch (KiCad schematic)
At the start: 4 parts, among them J5 Conn_01x02, J6 Conn_01x12

Commit message: merging. power stuff incomplete
Parts:
- R22: value R -> 0
Connections:
- net Battery Power: no longer J6.1 (Pin_1), J6.11 (Pin_11), J6.3 (Pin_3), J6.5 (Pin_5), J6.7 (Pin_7), J6.9 (Pin_9)
- net Pyro0/Armed Pyro: now also J6.1 (Pin_1), J6.11 (Pin_11), J6.3 (Pin_3), J6.5 (Pin_5), J6.7 (Pin_7), J6.9 (Pin_9)
Other:
- note added: "3.3V = (26V * R2)/(R1 + R2) 0.127 = R2 / (R1 + R2) -> 0.1 = R2 / (R1 + R2) R2 = 10k R1 = 90k (R2 + R1) = 100k V = IR 26V / 100k = 0.26mA Disarmed w/continuity = (3.3-0.7) * 0.1 = 0.26V Armed w/continuity = 26 * 0.1 = 2.6V"
- note removed: "PyroSense: Max Battery Voltage = 4S = 16.8V Logic Level = 3v3 3.3 >= 16.8(R2/(R1 + R2)) R2 = 10k R1 = 80k Vsense = 1.68V (max) Current (Max) = 16.8 / 90k = 0.187mA"
- moved on the sheet: R22
Changed lines of the file:
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@@
 	(generator_version "9.0")
 	(paper "A4")
-	(text "PyroSense:\nMax Battery Voltage = 4S = 16.8V\nLogic Level = 3v3\n\n3.3 >= 16.8(R2/(R1 + R2))\nR2 = 10k\nR1 = 80k\n\nVsense = 1.68V (max)\nCurrent (Max) = 16.8 / 90k = 0.187mA\n"
-		(exclude_from_sim no)
-		(at 228.346 22.352 0)
-		(effects
-			(font
-				(size 1.27 1.27)
-			)
-		)
-	)
 	(text "Arming Switch"
 		(exclude_from_sim no)
 		(at 97.536 50.8 0)
+		(effects
+			(font
+				(size 1.27 1.27)
+			)
+		)
+	)
+	(text "3.3V = (26V * R2)/(R1 + R2)\n0.127 = R2 / (R1 + R2)\n-> 0.1 = R2 / (R1 + R2)\nR2 = 10k\nR1 = 90k\n(R2 + R1) = 100k\n\nV = IR\n26V / 100k = 0.26mA\n\nDisarmed w/continuity = (3.3-0.7) * 0.1 = 0.26V\nArmed w/continuity = 26 * 0.1 = 2.6V\n"
+		(exclude_from_sim no)
+		(at 232.41 27.432 0)
 		(effects
 			(font
@@
 	)
 	(junction
+		(at 87.63 64.77)
+		(diameter 0)
+		(color 0 0 0 0)
+	)
+	(junction
 		(at 198.12 97.79)
 		(diameter 0)
@@
 	)
 	(junction
-		(at 87.63 62.23)
-		(diameter 0)
-		(color 0 0 0 0)
-	)
-	(junction
 		(at 201.93 80.01)
 		(diameter 0)
@@
 	)
 	(junction
-		(at 87.63 35.56)
+		(at 87.63 62.23)
 		(diameter 0)
 		(color 0 0 0 0)
@@
 	(wire
 		(pts
+			(xy 87.63 64.77) (xy 201.93 64.77)
+		)
+		(stroke
+			(width 0)
+			(type default)
+		)
+	)
+	(wire
+		(pts
 			(xy 201.93 92.71) (xy 198.12 92.71)
 		)
@@
 	(wire
 		(pts
+			(xy 87.63 64.77) (xy 87.63 74.93)
+		)
+		(stroke
+			(width 0)
+			(type default)
+		)
+	)
+	(wire
+		(pts
 			(xy 87.63 125.73) (xy 101.6 125.73)
 		)
@@
 	(wire
 		(pts
-			(xy 201.93 35.56) (xy 87.63 35.56)
-		)
-		(stroke
-			(width 0)
-			(type default)
-		)
-	)
-	(wire
-		(pts
 			(xy 130.81 99.06) (xy 142.24 99.06)
 		)
@@
 	(wire
 		(pts
+			(xy 57.15 34.29) (xy 57.15 40.64)
+		)
+		(stroke
+			(width 0)
+			(type default)
+		)
+	)
+	(wire
+		(pts
 			(xy 130.81 128.27) (xy 142.24 128.27)
 		)
@@
 	(wire
 		(pts
-			(xy 201.93 80.01) (xy 201.93 35.56)
-		)
-		(stroke
-			(width 0)
-			(type default)
-		)
-	)
-	(wire
-		(pts
 			(xy 130.81 104.14) (xy 142.24 104.14)
 		)
@@
 	(wire
 		(pts
+			(xy 57.15 48.26) (xy 57.15 50.8)
+		)
+		(stroke
+			(width 0)
+			(type default)
+		)
+	)
+	(wire
+		(pts
 			(xy 87.63 58.42) (xy 87.63 62.23)
 		)
@@
 	(wire
 		(pts
-			(xy 87.63 62.23) (xy 87.63 74.93)
+			(xy 87.63 62.23) (xy 87.63 64.77)
 		)
 		(stroke
@@
 	(wire
 		(pts
-			(xy 57.15 46.99) (xy 57.15 50.8)
-		)
-		(stroke
-			(width 0)
-			(type default)
-		)
-	)
-	(wire
-		(pts
-			(xy 87.63 31.75) (xy 87.63 35.56)
+			(xy 87.63 31.75) (xy 87.63 55.88)
 		)
 		(stroke
@@
 	(wire
 		(pts
-			(xy 57.15 34.29) (xy 57.15 39.37)
-		)
-		(stroke
-			(width 0)
-			(type default)
-		)
-	)
-	(wire
-		(pts
 			(xy 190.5 133.35) (xy 190.5 110.49)
 		)
@@
 	(wire
 		(pts
+			(xy 201.93 64.77) (xy 201.93 80.01)
+		)
+		(stroke
+			(width 0)
+			(type default)
+		)
+	)
+	(wire
+		(pts
 			(xy 130.81 74.93) (xy 142.24 74.93)
 		)
@@
 		(pts
 			(xy 198.12 102.87) (xy 198.12 97.79)
-		)
-		(stroke
-			(width 0)
-			(type default)
-		)
-	)
-	(wire
-		(pts
-			(xy 87.63 35.56) (xy 87.63 55.88)
 		)
 		(stroke
@@
 	(symbol
 		(lib_id "Device:R")
-		(at 57.15 43.18 0)
+		(at 57.15 44.45 0)
 		(unit 1)
 		(exclude_from_sim no)
@@
 		(fields_autoplaced yes)
 		(property "Reference" "R22"
-			(at 59.69 41.9099 0)
+			(at 59.69 43.1799 0)
 			(effects
 				(font
@@
 			)
 		)
-		(property "Value" "R"
-			(at 59.69 44.4499 0)
+		(property "Value" "0"
+			(at 59.69 45.7199 0)
 			(effects
 				(font
@@
 		)
 		(property "Footprint" ""
-			(at 55.372 43.18 90)
+			(at 55.372 44.45 90)
 			(effects
 				(font
@@
 		)
 		(property "Datasheet" "~"
-			(at 57.15 43.18 0)
+			(at 57.15 44.45 0)
 			(effects
 				(font
@@
 		)
 		(property "Description" "Resistor"
-			(at 57.15 43.18 0)
-			(effects
-				(font
+			(at 57.15 44.45 0)
+			(effects
+				(font

Commit message: schematic updates
Parts:
- R22: footprint (none) -> Resistor_SMD:R_0402_1005Metric
Changed lines of the file:
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@@
 			)
 		)
-		(property "Footprint" ""
+		(property "Footprint" "Resistor_SMD:R_0402_1005Metric"
 			(at 55.372 44.45 90)
 			(effects
