File: VoltV1/mcu.kicad_sch (KiCad schematic)
At the start: 25 parts, among them SW1 PTS810_SJM_250_SMTR_LFS, U1 ATSAMD51P20A-AUT, Y1 Crystal-32.768kHz

Commit message: merging. power stuff incomplete
Connections:
- net Barro1 CS: now also U1.39 (PB10); no longer U1.124 (PC31)
- net ICM Int1: now reaches U1.33 (PA08)
- net ICM20948 CS: now reaches U1.40 (PB11)
Changed lines of the file:
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@@
-	(wire
-		(pts
-			(xy 67.31 171.45) (xy 67.31 175.26)
-		)
-		(stroke
-			(width 0)
-			(type default)
-		)
-	)
 	(wire
 		(pts
@@
 	)
 	(label "VDDIO3.3"
-		(at 67.31 171.45 0)
+		(at 57.15 171.45 0)
 		(effects
 			(font
@@
 		)
 	)
+	(hierarchical_label "ICM20948 CS"
+		(shape input)
+		(at 154.94 100.33 0)
+		(effects
+			(font
+				(size 1.27 1.27)
+			)
+			(justify left)
+		)
+	)
 	(hierarchical_label "LED"
 		(shape input)
@@
 		)
 	)
+	(hierarchical_label "Barro1 CS"
+		(shape input)
+		(at 154.94 102.87 0)
+		(effects
+			(font
+				(size 1.27 1.27)
+			)
+			(justify left)
+		)
+	)
 	(hierarchical_label "Tx1"
 		(shape input)
@@
 		)
 	)
-	(hierarchical_label "Barro1 CS"
-		(shape input)
-		(at 257.81 44.45 0)
-		(effects
-			(font
+	(hierarchical_label "ICM Int1"
+		(shape input)
+		(at 154.94 118.11 0)
+		(effects
+			(font

Commit message: schematic updates
Parts:
- C10, C11, C12, C13, C14, C15, C16, C17, C18, C24, C25, C3, C4, C5, C6, C7, C8, C9: footprint Capacitor_SMD:C_0603_1608Metric -> Capacitor_SMD:C_0402_1005Metric
- R3, R5: footprint Resistor_SMD:R_0603_1608Metric -> Resistor_SMD:R_0402_1005Metric
