File: VoltV1/sensors.kicad_sch (KiCad schematic)
At the start: 10 parts, among them U4 MS5607-02BA, U5 MS5607-02BA, U7 ICM-20948, U8 LSM6DSV320XTR

Commit message: merging. power stuff incomplete
Parts:
- added C26, C51, C54, C55, C56, C57, C58: 0.1uF, symbol Device:C
- added R27, R29, R30, R37, R38: 100k, Resistor_SMD:R_0603_1608Metric, symbol Device:R_Small
- added R32, R33, R34: 100, Resistor_SMD:R_0603_1608Metric, symbol Device:R_Small
- added U17, U18, U19: SN74LVC2T45, Package_BGA:Texas_DSBGA-8_0.9x1.9mm_Layout2x4_P0.5mm, symbol VOLTV1:SN74LVC2T45
Connections:
- net +1V8: now also U7.8 (VDDIO), C26.1, C54.1, C56.1, C58.2, R38.2, U17.A1 (VCCA), U18.A1 (VCCA), U19.A2 (VCCB)
- net +3.3V: now also C51.1, C55.1, C57.1, U17.A2 (VCCB), U18.A2 (VCCB), U19.A1 (VCCA)
- net Barro0 CS: now also R30.1
- net Barro1 CS: now also R29.1
- net GND: now also U7.20 (RESV_GND), C26.2, C51.2, C54.2, C55.2, C56.2, C57.2, C58.1, U17.D1 (GND), U17.D2 (DIR), U18.D1 (GND), U18.D2 (DIR), U19.D1 (GND), U19.D2 (DIR)
- net LSM CS: now also R27.1
- net Miso0: now also R32.2; no longer U8.1 (SDO/TA0)
- net Miso1: now also U19.B1 (A1)
- net Mosi0: now also R34.2; no longer U8.14 (SDA)
- net Mosi1: now also U18.C2 (B2)
- net Sck0: now also R33.1; no longer U8.13 (SCL)
- net Sck1: now also U18.B2 (B1)
- net ICM Int1: now reaches U7.12 (INT1)
- net at U7.22 (nCS): now also R38.1, U17.B1 (A1)
- net at U7.23 (SCL/SCLK): now also U18.B1 (A1)
- net at U7.24 (SDA/SDI): now also U18.C1 (A2)
- net at U7.9 (SDO/AD0): now also U19.B2 (B1)
- new net: R32.1, U8.1 (SDO/TA0)
- new net: R33.2, U8.13 (SCL)
- new net: R34.1, U8.14 (SDA)
- new net +3V3: R27.2, R29.2, R30.2, R37.1
- new net ICM20948 CS: R37.2, U17.B2 (B1)
- no-connect marks 3 -> 8
Other:
- note added: "B (mcu) -> A (sensor)"
- note added: "B (sensor) -> A (mcu)"
- note added: "DOUBLE CHECK THESE PULLUPS ON CS"
- note added: "These are flipped from others as we want 1v8 -> 3v3"
- moved on the sheet: C1, C19, C2, C20, C53, U4, U5, U8

Commit message: updates to schematic
Connections:
- no-connect marks 8 -> 9
Changed lines of the file:
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@@
+	)
+	(no_connect
+		(at 193.04 58.42)
 	)
 	(no_connect

Commit message: schematic updates
Parts:
- C1, C19, C2, C20: footprint Capacitor_SMD:C_0603_1608Metric -> Capacitor_SMD:C_0402_1005Metric
- C26, C51, C52, C53, C54, C55, C56, C57, C58: footprint (none) -> Capacitor_SMD:C_0402_1005Metric
- R27, R29, R30, R32, R33, R34, R37, R38: footprint Resistor_SMD:R_0603_1608Metric -> Resistor_SMD:R_0402_1005Metric
Changed lines of the file:
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@@
 			)
 		)
-		(property "Footprint" "Resistor_SMD:R_0603_1608Metric"
+		(property "Footprint" "Resistor_SMD:R_0402_1005Metric"
 			(at 120.65 139.7 0)
 			(effects
@@
 			)
 		)
-		(property "Footprint" "Resistor_SMD:R_0603_1608Metric"
+		(property "Footprint" "Resistor_SMD:R_0402_1005Metric"
 			(at 205.74 105.41 0)
 			(effects
@@
 			)
 		)
-		(property "Footprint" "Capacitor_SMD:C_0603_1608Metric"
+		(property "Footprint" "Capacitor_SMD:C_0402_1005Metric"
 			(at 100.0252 165.1 0)
 			(effects
@@
 			)
 		)
-		(property "Footprint" "Resistor_SMD:R_0603_1608Metric"
+		(property "Footprint" "Resistor_SMD:R_0402_1005Metric"
 			(at 101.6 137.16 0)
 			(effects
@@
 			)
 		)
-		(property "Footprint" "Capacitor_SMD:C_0603_1608Metric"
+		(property "Footprint" "Capacitor_SMD:C_0402_1005Metric"
 			(at 137.4648 39.37 0)
 			(effects
@@
 			)
 		)
-		(property "Footprint" ""
+		(property "Footprint" "Capacitor_SMD:C_0402_1005Metric"
 			(at 173.6852 121.92 0)
 			(effects
@@
 			)
 		)
-		(property "Footprint" ""
+		(property "Footprint" "Capacitor_SMD:C_0402_1005Metric"
 			(at 174.2948 43.18 0)
 			(effects
@@
 			)
 		)
-		(property "Footprint" ""
+		(property "Footprint" "Capacitor_SMD:C_0402_1005Metric"
 			(at 121.6152 85.09 0)
 			(effects
@@
 			)
 		)
-		(property "Footprint" ""
+		(property "Footprint" "Capacitor_SMD:C_0402_1005Metric"
 			(at 115.2652 85.09 0)
 			(effects
@@
 			)
 		)
-		(property "Footprint" ""
+		(property "Footprint" "Capacitor_SMD:C_0402_1005Metric"
 			(at 232.1052 106.68 0)
 			(effects
@@
 			)
 		)
-		(property "Footprint" ""
+		(property "Footprint" "Capacitor_SMD:C_0402_1005Metric"
 			(at 270.2052 40.64 0)
 			(effects
@@
 			)
 		)
-		(property "Footprint" "Resistor_SMD:R_0603_1608Metric"
+		(property "Footprint" "Resistor_SMD:R_0402_1005Metric"
 			(at 219.71 124.46 0)
 			(effects
@@
 			)
 		)
-		(property "Footprint" "Resistor_SMD:R_0603_1608Metric"
+		(property "Footprint" "Resistor_SMD:R_0402_1005Metric"
 			(at 104.14 29.21 0)
 			(effects
@@
 			)
 		)
-		(property "Footprint" "Capacitor_SMD:C_0603_1608Metric"
+		(property "Footprint" "Capacitor_SMD:C_0402_1005Metric"
 			(at 77.7748 43.18 0)
 			(effects
@@
 			)
 		)
-		(property "Footprint" ""
+		(property "Footprint" "Capacitor_SMD:C_0402_1005Metric"
 			(at 167.3352 121.92 0)
 			(effects
@@
 			)
 		)
-		(property "Footprint" "Resistor_SMD:R_0603_1608Metric"
+		(property "Footprint" "Resistor_SMD:R_0402_1005Metric"
 			(at 43.18 142.24 0)
 			(effects
@@
 			)
 		)
-		(property "Footprint" "Capacitor_SMD:C_0603_1608Metric"
+		(property "Footprint" "Capacitor_SMD:C_0402_1005Metric"
 			(at 25.7048 152.4 0)
 			(effects
@@
 			)
 		)
-		(property "Footprint" ""
+		(property "Footprint" "Capacitor_SMD:C_0402_1005Metric"
 			(at 179.3748 62.23 0)
 			(effects
@@
 			)
 		)
-		(property "Footprint" ""
+		(property "Footprint" "Capacitor_SMD:C_0402_1005Metric"
 			(at 238.4552 106.68 0)
 			(effects
@@
 			)
 		)
-		(property "Footprint" "Resistor_SMD:R_0603_1608Metric"
+		(property "Footprint" "Resistor_SMD:R_0402_1005Metric"
 			(at 35.56 30.48 0)
 			(effects
@@
 			)
 		)
-		(property "Footprint" "Resistor_SMD:R_0603_1608Metric"
+		(property "Footprint" "Resistor_SMD:R_0402_1005Metric"
 			(at 104.14 144.78 0)
 			(effects
