File: VoltV1/storage.kicad_sch (KiCad schematic)
At the start: 8 parts, among them U2 S25FL512SAGMF, U6 MB85RS64V

Commit message: merging. power stuff incomplete
Parts:
- added R31: 100k, Resistor_SMD:R_0603_1608Metric, symbol Device:R_Small
Connections:
- net +3.3V: now also R31.2
- net FRAM CS: now also R31.1
Changed lines of the file:
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@@
+	)
+	(junction
+		(at 176.53 59.69)
+		(diameter 0)
+		(color 0 0 0 0)
 	)
 	(junction
@@
 		(color 0 0 0 0)
 	)
+	(junction
+		(at 176.53 71.12)
+		(diameter 0)
+		(color 0 0 0 0)
+	)
 	(no_connect
 		(at 78.74 72.39)
@@
 	(wire
 		(pts
-			(xy 157.48 59.69) (xy 186.69 59.69)
+			(xy 157.48 59.69) (xy 176.53 59.69)
+		)
+		(stroke
+			(width 0)
+			(type default)
+		)
+	)
+	(wire
+		(pts
+			(xy 172.72 67.31) (xy 172.72 71.12)
 		)
 		(stroke
@@
 	(wire
 		(pts
+			(xy 176.53 59.69) (xy 176.53 62.23)
+		)
+		(stroke
+			(width 0)
+			(type default)
+		)
+	)
+	(wire
+		(pts
+			(xy 167.64 67.31) (xy 172.72 67.31)
+		)
+		(stroke
+			(width 0)
+			(type default)
+		)
+	)
+	(wire
+		(pts
 			(xy 186.69 53.34) (xy 186.69 59.69)
 		)
@@
 	(wire
 		(pts
+			(xy 176.53 71.12) (xy 177.8 71.12)
+		)
+		(stroke
+			(width 0)
+			(type default)
+		)
+	)
+	(wire
+		(pts
+			(xy 176.53 59.69) (xy 186.69 59.69)
+		)
+		(stroke
+			(width 0)
+			(type default)
+		)
+	)
+	(wire
+		(pts
 			(xy 116.84 60.96) (xy 116.84 69.85)
 		)
@@
 	(wire
 		(pts
+			(xy 172.72 71.12) (xy 176.53 71.12)
+		)
+		(stroke
+			(width 0)
+			(type default)
+		)
+	)
+	(wire
+		(pts
 			(xy 168.91 81.28) (xy 168.91 78.74)
 		)
@@
 		(pts
 			(xy 67.31 80.01) (xy 78.74 80.01)
+		)
+		(stroke
+			(width 0)
+			(type default)
+		)
+	)
+	(wire
+		(pts
+			(xy 176.53 67.31) (xy 176.53 71.12)
 		)
 		(stroke
@@
 	(hierarchical_label "FRAM CS"
 		(shape input)
-		(at 177.8 71.12 180)
+		(at 167.64 67.31 180)
 		(effects
 			(font
@@
 	)
 	(symbol
+		(lib_id "Device:R_Small")
+		(at 176.53 64.77 180)
+		(unit 1)
+		(exclude_from_sim no)
+		(in_bom yes)
+		(on_board yes)
+		(dnp no)
+		(property "Reference" "R31"
+			(at 172.72 60.96 0)
+			(effects
+				(font
+					(size 1.27 1.27)
+				)
+			)
+		)
+		(property "Value" "100k"
+			(at 172.72 63.5 0)
+			(effects
+				(font
+					(size 1.27 1.27)
+				)
+			)
+		)
+		(property "Footprint" "Resistor_SMD:R_0603_1608Metric"
+			(at 176.53 64.77 0)
+			(effects
+				(font
+					(size 1.27 1.27)
+				)
+				(hide yes)
+			)
+		)
+		(property "Datasheet" "~"
+			(at 176.53 64.77 0)
+			(effects
+				(font
+					(size 1.27 1.27)
+				)
+				(hide yes)
+			)
+		)
+		(property "Description" ""
+			(at 176.53 64.77 0)
+			(effects
+				(font
+					(size 1.27 1.27)
+				)
+			)
+		)
+		(property "LCSC" "C25077"
+			(at 176.53 64.77 90)
+			(effects
+				(font
+					(size 1.27 1.27)
+				)
+				(hide yes)
+			)
+		)
+		(pin "1"
+		)
+		(pin "2"
+		)
+		(instances
+			(project "VoltV1"
+				(path "/4dc02877-6404-4472-a9f6-00d826e215ba/f67f1027-daba-493a-8bee-d229304ca6b6"
+					(reference "R31")
+					(unit 1)
+				)
+			)
+		)
+	)
+	(symbol
 		(lib_id "power:GND")
 		(at 121.92 85.09 0)
@@
 			)
 		)
-		(property "Datasheet" ""
+		(property "Datasheet" "https://www.ramxeed.com/assets/images/products/datasheet/FeRAM/s4/MB85RS64V-DS6v1-E.pdf"
 			(at 190.5 76.2 0)
 			(effects

Commit message: updates to schematic
Parts:
- U6: value MB85RS64V -> MB85RS64
Other:
- note added: "MB85RS64PNF-G-JNE1"
- note removed: "FRAM Datasheet"
Changed lines of the file:
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@@
 	(generator_version "9.0")
 	(paper "A4")
-	(text "FRAM Datasheet"
-		(exclude_from_sim no)
-		(at 190.246 85.09 0)
-		(effects
-			(font
-				(size 1.27 1.27)
-			)
-			(href "https://www.ramxeed.com/assets/images/products/datasheet/FeRAM/s4/MB85RS64V-DS6v1-E.pdf")
-		)
-	)
 	(text "Internal pullup on WP and Reset\n"
 		(exclude_from_sim no)
@@
 			)
 			(href "https://mm.digikey.com/Volume0/opasdata/d220001/medias/docus/7130/001-98284%20Rev%20U.pdf")
+		)
+	)
+	(text "MB85RS64PNF-G-JNE1\n"
+		(exclude_from_sim no)
+		(at 191.008 84.582 0)
+		(effects
+			(font
+				(size 1.27 1.27)
+			)
 		)
 	)
@@
 			)
 		)
-		(property "Value" "MB85RS64V"
+		(property "Value" "MB85RS64"
 			(at 190.5 66.04 0)
 			(effects

Commit message: schematic updates
Parts:
- C21, C22, C23: footprint Capacitor_SMD:C_0603_1608Metric -> Capacitor_SMD:C_0402_1005Metric
- R31, R4, R6, R7: footprint Resistor_SMD:R_0603_1608Metric -> Resistor_SMD:R_0402_1005Metric
Changed lines of the file:
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@@
 			)
 		)
-		(property "Footprint" "Resistor_SMD:R_0603_1608Metric"
+		(property "Footprint" "Resistor_SMD:R_0402_1005Metric"
 			(at 210.312 69.85 90)
 			(effects
@@
 			)
 		)
-		(property "Footprint" "Resistor_SMD:R_0603_1608Metric"
+		(property "Footprint" "Resistor_SMD:R_0402_1005Metric"
 			(at 176.53 64.77 0)
 			(effects
@@
 			)
 		)
-		(property "Footprint" "Capacitor_SMD:C_0603_1608Metric"
+		(property "Footprint" "Capacitor_SMD:C_0402_1005Metric"
 			(at 113.9952 77.47 0)
 			(effects
@@
 			)
 		)
-		(property "Footprint" "Resistor_SMD:R_0603_1608Metric"
+		(property "Footprint" "Resistor_SMD:R_0402_1005Metric"
 			(at 155.702 72.39 90)
 			(effects
@@
 			)
 		)
-		(property "Footprint" "Capacitor_SMD:C_0603_1608Metric"
+		(property "Footprint" "Capacitor_SMD:C_0402_1005Metric"
 			(at 214.63 58.7248 0)
 			(effects
@@
 			)
 		)
-		(property "Footprint" "Resistor_SMD:R_0603_1608Metric"
+		(property "Footprint" "Resistor_SMD:R_0402_1005Metric"
 			(at 59.69 81.788 90)
 			(effects
@@
 			)
 		)
-		(property "Footprint" "Capacitor_SMD:C_0603_1608Metric"
+		(property "Footprint" "Capacitor_SMD:C_0402_1005Metric"
 			(at 64.77 62.5348 0)
 			(effects
