File: VoltV1/VoltV1.kicad_pcb (KiCad board)
At the start: 2 copper layers, 62 parts, among them J1 USBC, J2 SFM-120-02-X-D-A, J3 Conn_Coaxial, J4 Conn_Coaxial, SW1 PTS810_SJM_250_SMTR_LFS, U1 ATSAMD51P20A-AUT, U2 S25FL512SAGMF, U3 MAX-M10S-00B, U4 MS5607-02BA, U5 MS5607-02BA, U6 MB85RS64V, U7 ICM-20948, U8 LSM6DSV320XTR, U9 E22-900M30S, Y1 Crystal-32.768kHz

Commit message: updates to schematic
Parts:
- removed C26: 1nF, Capacitor_SMD:C_0603_1608Metric
- removed the D1 at (171.1, 137.5)
- removed the D1 at (119.0, 149.2)
- removed J3, J4: Conn_Coaxial, Connector_Coaxial:SMA_Molex_73251-1153_EdgeMount_Horizontal
- removed the R18 at (119.0, 151.8)
- removed the R18 at (168.6, 137.4)
- removed U9: E22-900M30S, VOLTV1:XCVR_E22-900M30S
- added C64: 100n, Capacitor_SMD:C_0603_1608Metric, F.Cu at (138.9, 93.7)
- added C65: 100n, Capacitor_SMD:C_0603_1608Metric, F.Cu at (138.9, 96.2)
- added C66: 47n, Capacitor_SMD:C_0603_1608Metric, F.Cu at (142.9, 86.1)
- added C67: 1u, Capacitor_SMD:C_0603_1608Metric, F.Cu at (142.9, 88.6)
- added C68: 47p, Capacitor_SMD:C_0402_1005Metric, F.Cu at (156.4, 74.6)
- added C69: 47p, Capacitor_SMD:C_0402_1005Metric, F.Cu at (156.4, 76.6)
- added C70: 1n, Capacitor_SMD:C_0603_1608Metric, F.Cu at (142.9, 91.2)
- added C71: 1n, Capacitor_SMD:C_0603_1608Metric, F.Cu at (142.9, 93.7)
- added C72: 47p, Capacitor_SMD:C_0402_1005Metric, F.Cu at (156.4, 78.5)
- added D1: LED, LED_SMD:LED_0603_1608Metric, F.Cu at (162.5, 145.3)
- added D3: D_Schottky, Diode_SMD:D_SOD-123, F.Cu at (170.0, 138.1)
- added D7: SS1F4-M3/H, Diode_SMD:D_SOD-123, F.Cu at (162.8, 101.7)
- added D8: LED, LED_SMD:LED_0603_1608Metric, F.Cu at (161.9, 90.0)
- added FL1: 0900FM15K0039, RF_Converter:Balun_Johanson_0900FM15K0039, F.Cu at (150.7, 93.3)
- added J7: Conn_01x08, Connector_JST:JST_GH_BM08B-GHS-TBT_1x08-1MP_P1.25mm_Vertical, F.Cu at (164.2, 132.6)
- added J9: Conn_Coaxial, Connector_Coaxial:SMA_Molex_73251-1153_EdgeMount_Horizontal, F.Cu at (151.7, 78.3)
- added LS1: CMT-0525-75-SMT-TR, VOLTV1:XDCR_CMT-0525-75-SMT-TR, F.Cu at (163.8, 140.2)
- added Q1: STL66DN3LLH5, VOLTV1:POWERFLAT5X6_STL66_STM, F.Cu at (149.2, 136.2)
- added Q2: STL66DN3LLH5, VOLTV1:POWERFLAT5X6_STL66_STM, F.Cu at (203.2, 122.5)
- added Q3: STL66DN3LLH5, VOLTV1:POWERFLAT5X6_STL66_STM, F.Cu at (138.3, 136.2)
- added Q4: IRLML6244, Package_TO_SOT_SMD:SOT-23, F.Cu at (169.5, 142.2)
- added Q5: CSD18563Q5A, Package_TO_SOT_SMD:TDSON-8-1, F.Cu at (189.6, 143.2)
- added Q6: SI3421DV-T1-GE3, Package_SO:TSOP-6_1.65x3.05mm_P0.95mm, F.Cu at (164.2, 95.9)
- added R18: 270, Resistor_SMD:R_0603_1608Metric, F.Cu at (158.5, 137.7)
- added R23: 2k, Resistor_SMD:R_0603_1608Metric, F.Cu at (158.5, 140.2)
- added R24: 100k, Resistor_SMD:R_0603_1608Metric, F.Cu at (158.5, 142.7)
- added R25: 50, Resistor_SMD:R_0603_1608Metric, F.Cu at (158.5, 145.2)
- added R26: 100k, Resistor_SMD:R_0603_1608Metric, F.Cu at (181.6, 89.2)
- added R27: 100k, Resistor_SMD:R_0603_1608Metric, F.Cu at (162.5, 111.2)
- added R29: 100k, Resistor_SMD:R_0603_1608Metric, F.Cu at (162.5, 113.7)
- added R30: 100k, Resistor_SMD:R_0603_1608Metric, F.Cu at (162.5, 116.2)
- added R31: 100k, Resistor_SMD:R_0603_1608Metric, F.Cu at (182.0, 135.3)
- added R32: 100, Resistor_SMD:R_0603_1608Metric, F.Cu at (162.5, 118.7)
- added R33: 100, Resistor_SMD:R_0603_1608Metric, F.Cu at (166.5, 111.2)
- added R34: 100, Resistor_SMD:R_0603_1608Metric, F.Cu at (166.5, 113.7)
- added R35: 100k, Resistor_SMD:R_0603_1608Metric, F.Cu at (167.6, 101.2)
- added R36: 10k, Resistor_SMD:R_0603_1608Metric, F.Cu at (146.9, 86.1)
- added R37: 100k, Resistor_SMD:R_0603_1608Metric, F.Cu at (166.5, 116.2)
- added R38: 100k, Resistor_SMD:R_0603_1608Metric, F.Cu at (166.5, 118.7)
- added R39: 220R, Resistor_SMD:R_0402_1005Metric, F.Cu at (150.4, 96.4)
- added R40: 220R, Resistor_SMD:R_0603_1608Metric, F.Cu at (146.9, 88.6)
- added R41: 100R, Resistor_SMD:R_0603_1608Metric, F.Cu at (146.9, 91.2)
- added U10: LM5050-1, Package_TO_SOT_SMD:TSOT-23-6, F.Cu at (182.9, 142.3)
- added U11: AP63205WU, Package_TO_SOT_SMD:TSOT-23-6, F.Cu at (182.9, 146.9)
- added U12: TPD2EUSB30, Package_TO_SOT_SMD:Texas_DRT-3, F.Cu at (144.6, 129.2)
- added U13: MIC5528-3.3YMT-TR, VOLTV1:SON40P120X120X60-7N, F.Cu at (187.6, 148.0)
- added U14: MIC5528-3.3YMT-TR, VOLTV1:SON40P120X120X60-7N, F.Cu at (187.6, 150.8)
- added U15: SAM-M8Q, RF_GPS:ublox_SAM-M8Q, F.Cu at (168.6, 80.2)
- added U16: TMCS1108A2B, Package_SO:SOIC-8_3.9x4.9mm_P1.27mm, F.Cu at (147.3, 124.7)
- added U17: SN74LVC2T45, Package_BGA:Texas_DSBGA-8_0.9x1.9mm_Layout2x4_P0.5mm, F.Cu at (158.5, 122.5)
- added U18: SN74LVC2T45, Package_BGA:Texas_DSBGA-8_0.9x1.9mm_Layout2x4_P0.5mm, F.Cu at (162.5, 122.5)
- added U19: SN74LVC2T45, Package_BGA:Texas_DSBGA-8_0.9x1.9mm_Layout2x4_P0.5mm, F.Cu at (166.5, 122.5)
- added U20: ~, Package_SO:SOIC-8_3.9x4.9mm_P1.27mm, F.Cu at (149.0, 143.1)
- added U21: ~, Package_SO:SOIC-8_3.9x4.9mm_P1.27mm, F.Cu at (203.0, 129.4)
- added U22: ~, Package_SO:SOIC-8_3.9x4.9mm_P1.27mm, F.Cu at (138.1, 143.1)
- C27: value .1uF -> 10p; footprint Capacitor_SMD:C_0603_1608Metric -> Capacitor_SMD:C_0402_1005Metric
- C28: value .1uF -> 100n
- C29: value 10uF -> 100n
- C32: value 10nF -> 47n
- L3: value 27n -> 47n
- R8: value 10 -> 270
- U3: value MAX-M10S-00B -> SX1262IMLTRT; footprint VOLTV1:XCVR_MAX-M10S-00B -> Package_DFN_QFN:QFN-24-1EP_4x4mm_P0.5mm_EP2.6x2.6mm
- moved C30 122.9 mm to (181.6, 76.7)
- moved C31 122.9 mm to (181.6, 79.2)
- moved R8 107.1 mm to (165.9, 90.0)
- moved Y1 94.9 mm to (204.2, 93.9), turned to 0 degrees
- moved C27 88.0 mm to (156.4, 72.6)
- moved C24 83.3 mm to (195.7, 98.7), turned to 0 degrees
- moved L3 82.5 mm to (142.9, 96.2)
- moved C10 81.3 mm to (191.6, 91.2)
- moved C11 81.3 mm to (191.6, 93.7)
- moved C9 81.3 mm to (191.6, 88.7)
- moved C25 80.8 mm to (195.7, 101.2), turned to 0 degrees
- moved C3 80.8 mm to (187.6, 88.7)
- moved C4 80.8 mm to (187.6, 91.2)
- moved C5 80.8 mm to (187.6, 93.7)
- moved C6 80.8 mm to (187.6, 96.2)
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Connections:
- net /mcu/ArmCont renamed /Pyros/PyroSense3
- net /mcu/RESETN renamed /IO/RESETN
- C27 pad 1: +5V -> Net-(C27-Pad1)
- C27 pad 2: GND -> Net-(Y2-OUTPUT)
- C28 pad 1: +5V -> +3.3V
- C29 pad 1: +5V -> +3.3V
- C32 pad 2: Net-(C32-Pad2) -> /GPSRadio/Radio/VR_PA
- J1 pad A4: unconnected-(J1-VBUS-PadA4) -> /power/VUSB
- J1 pad A6: Net-(J1-DP1) -> /mcu/D+
- J1 pad A7: Net-(J1-DN1) -> /mcu/D-
- J1 pad A9: unconnected-(J1-VBUS__1-PadA9) -> /power/VUSB
- J1 pad B4: unconnected-(J1-VBUS__2-PadB4) -> /power/VUSB
- J1 pad B6: Net-(J1-DP1) -> /mcu/D+
- J1 pad B7: Net-(J1-DN1) -> /mcu/D-
- J1 pad B9: unconnected-(J1-VBUS__3-PadB9) -> /power/VUSB
- J1 pad S1: Net-(J1-SHELL) -> GND
- J1 pad S2: Net-(J1-SHELL) -> GND
- J1 pad S3: Net-(J1-SHELL) -> GND
- J1 pad S4: Net-(J1-SHELL) -> GND
- J2 pad 01: unconnected-(J2-Pad01) -> /daughterInterface/Daughter Battery
- J2 pad 02: unconnected-(J2-Pad02) -> /daughterInterface/Daughter 5V
- J2 pad 03: unconnected-(J2-Pad03) -> /daughterInterface/Daughter Battery
- J2 pad 04: unconnected-(J2-Pad04) -> /daughterInterface/Daughter 5V
- J2 pad 05: unconnected-(J2-Pad05) -> /daughterInterface/Daughter Battery
- J2 pad 06: unconnected-(J2-Pad06) -> /daughterInterface/Daughter 3.3V
- J2 pad 16: /daughterInterface/DaughterAnalogue7 -> /daughterInterface/DaughterGPIO7
- J2 pad 18: /daughterInterface/DaughterAnalogue8 -> /daughterInterface/DaughterGPIO8
- J2 pad 20: /daughterInterface/DaughterAnalogue9 -> /daughterInterface/DaughterGPIO9
- L3 pad 1: Net-(C32-Pad2) -> /GPSRadio/Radio/VR_PA
- L3 pad 2: Net-(J3-In) -> /GPSRadio/Radio/RFO
- R4 pad 2: /storage/Flash CS -> /mcu/Flash CS
- R8 pad 1: Net-(U3-VCC_RF) -> Net-(U15-TIMEPULSE)
- R8 pad 2: Net-(C32-Pad2) -> Net-(D8-A)
- U1 pad 119: /mcu/SWCLK -> /IO/SWCLK
- U1 pad 12: /daughterInterface/DaughterAnalogue7 -> /Pyros/PyroSense0
- U1 pad 120: /mcu/SWDIO -> /IO/SWDIO
- U1 pad 122: unconnected-(U1B-PB31-Pad122) -> /mcu/LSM Int 1
- U1 pad 123: unconnected-(U1B-PC30-Pad123) -> /mcu/LSM CS
- U1 pad 125: /mcu/PyroPWM4 -> /Pyros/PyroPWM4
- U1 pad 127: unconnected-(U1B-PB02-Pad127) -> /mcu/Barro0 CS
- U1 pad 19: unconnected-(U1A-PB08-Pad19) -> /Pyros/PyroSense4
- U1 pad 20: unconnected-(U1A-PB09-Pad20) -> /Pyros/PyroSense5
- U1 pad 27: /mcu/GPIOspare0 -> /daughterInterface/DaughterGPIO7
- U1 pad 28: /mcu/GPIOspare1 -> /daughterInterface/DaughterGPIO8
- U1 pad 3: /daughterInterface/DaughterAnalogue8 -> /Pyros/PyroSense1
- U1 pad 33: /mcu/PyroGPIO2 -> /mcu/ICM Int1
- U1 pad 34: /mcu/PyroGPIO3 -> unconnected-(U1A-PA09-Pad34)
- U1 pad 35: /mcu/PyroGPIO4 -> unconnected-(U1A-PA10-Pad35)
- U1 pad 36: /mcu/PyroGPIO5 -> unconnected-(U1A-PA11-Pad36)
- U1 pad 39: /mcu/PyroGPIO0 -> /mcu/Barro1 CS
- U1 pad 4: /daughterInterface/DaughterAnalogue9 -> /Pyros/PyroSense2
- U1 pad 40: /mcu/PyroGPIO1 -> /mcu/ICM20948 CS
- U1 pad 49: unconnected-(U1A-PD10-Pad49) -> /mcu/Flash CS
- U1 pad 51: /mcu/GPIOspare2 -> /daughterInterface/DaughterGPIO9
- U1 pad 52: unconnected-(U1A-PC10-Pad52) -> /GPSRadio/TxEN Radio
- U1 pad 55: unconnected-(U1A-PC11-Pad55) -> /GPSRadio/RxEn Radio
- U1 pad 56: unconnected-(U1A-PC12-Pad56) -> /GPSRadio/CS Radio
- U1 pad 57: unconnected-(U1A-PC13-Pad57) -> /GPSRadio/Reset Radio
- U1 pad 58: unconnected-(U1A-PC14-Pad58) -> /GPSRadio/Dio1 Radio
- U1 pad 59: unconnected-(U1A-PC15-Pad59) -> /GPSRadio/Busy Radio
- U1 pad 63: /mcu/PyroPWM5 -> /Pyros/PyroPWM5
- U1 pad 66: unconnected-(U1B-PA16-Pad66) -> /mcu/LSM Int 2
- U1 pad 67: unconnected-(U1B-PA17-Pad67) -> /mcu/Hold Flash
- U1 pad 74: /mcu/PyroPWM0 -> /Pyros/PyroPWM0
- U1 pad 75: /mcu/PyroPWM1 -> /Pyros/PyroPWM1
- U1 pad 82: unconnected-(U1B-PB16-Pad82) -> /mcu/FRAM CS
- U1 pad 93: /mcu/Buzzer -> /IO/Buzzer
- U1 pad 98: /mcu/PyroPWM2 -> /Pyros/PyroPWM2
- U1 pad 99: /mcu/PyroPWM3 -> /Pyros/PyroPWM3
- U2 pad 1: /storage/Hold Flash -> /mcu/Hold Flash
- U2 pad 7: /storage/Flash CS -> /mcu/Flash CS
- U3 pad 1: GND -> +3.3V
- U3 pad 10: GND -> +3.3V
- U3 pad 11: Net-(J3-In) -> +3.3V
- U3 pad 12: GND -> /GPSRadio/Radio/DIO2
- U3 pad 13: unconnected-(U3-LNA_EN-Pad13) -> /GPSRadio/Radio/DIO1
- U3 pad 14: Net-(U3-VCC_RF) -> /GPSRadio/Radio/BUSY_RF
- U3 pad 15: unconnected-(U3-VIO_SEL-Pad15) -> /GPSRadio/Reset Radio
- U3 pad 16: unconnected-(U3-SDA-Pad16) -> /GPSRadio/Radio/MISO
- U3 pad 17: unconnected-(U3-SCL-Pad17) -> /GPSRadio/Radio/MOSI
- U3 pad 18: unconnected-(U3-~{SAFEBOOT}-Pad18) -> /GPSRadio/Radio/SCK
- U3 pad 2: /GPSRadio/TxGPS -> GND
- U3 pad 3: /GPSRadio/RxGPS -> /GPSRadio/Radio/XTA
- U3 pad 5: unconnected-(U3-EXTINT-Pad5) -> GND
- U3 pad 7: GND -> /GPSRadio/Radio/VREG
- U4 pad 4: /sensors/Barro1 CS -> /mcu/Barro1 CS
- U5 pad 4: /sensors/Barro0 CS -> /mcu/Barro0 CS
- U6 pad 1: /storage/FRAM CS -> /mcu/FRAM CS
- U7 pad 10: unconnected-(U7-REGOUT-Pad10) -> Net-(U7-REGOUT)
- U7 pad 12: unconnected-(U7-INT1-Pad12) -> /mcu/ICM Int1
- U7 pad 13: unconnected-(U7-VDD-Pad13) -> +1V8
- U7 pad 20: unconnected-(U7-RESV_GND-Pad20) -> GND
- U7 pad 22: unconnected-(U7-nCS-Pad22) -> Net-(U17-A1)
- U7 pad 23: unconnected-(U7-SCL/SCLK-Pad23) -> Net-(U18-A1)
- U7 pad 24: unconnected-(U7-SDA/SDI-Pad24) -> Net-(U18-A2)
- U7 pad 8: unconnected-(U7-VDDIO-Pad8) -> +1V8
- U7 pad 9: unconnected-(U7-SDO/AD0-Pad9) -> Net-(U19-B1)
- U8 pad 1: /mcu/Miso0 -> Net-(U8-SDO/TA0)
- U8 pad 12: /sensors/LSM CS -> /mcu/LSM CS
- U8 pad 13: /mcu/Sck0 -> Net-(U8-SCL)
- U8 pad 14: /mcu/Mosi0 -> Net-(U8-SDA)
- U8 pad 4: /sensors/LSM Int 1 -> /mcu/LSM Int 1
- U8 pad 9: /sensors/LSM Int 2 -> /mcu/LSM Int 2
Other:
- board text removed: "Flash"

Commit message: schematic updates
Parts:
- added C26: 0.1uF, Capacitor_SMD:C_0402_1005Metric, F.Cu at (265.3, 20.0)
- added C33: 1nF, Capacitor_SMD:C_0402_1005Metric, F.Cu at (126.0, 180.4)
- added C34: 1nF, Capacitor_SMD:C_0402_1005Metric, F.Cu at (126.0, 182.4)
- added C35: 10uF, Capacitor_SMD:C_0402_1005Metric, F.Cu at (126.0, 184.3)
- added C36: 1uF, Capacitor_SMD:C_0402_1005Metric, F.Cu at (30.4, 162.5)
- added C37: .1uF, Capacitor_SMD:C_0402_1005Metric, F.Cu at (126.0, 186.3)
- added C38: 0.1uF, Capacitor_SMD:C_0402_1005Metric, F.Cu at (30.4, 164.5)
- added C39: 1nF, Capacitor_SMD:C_0402_1005Metric, F.Cu at (110.5, 180.4)
- added C40: 1nF, Capacitor_SMD:C_0402_1005Metric, F.Cu at (110.5, 182.4)
- added C41: 10uF, Capacitor_SMD:C_0402_1005Metric, F.Cu at (110.5, 184.3)
- added C42: 22uF, Capacitor_SMD:C_0402_1005Metric, F.Cu at (30.4, 166.4)
- added C43: .1uF, Capacitor_SMD:C_0402_1005Metric, F.Cu at (110.5, 186.3)
- added C44: 10uF, Capacitor_SMD:C_0402_1005Metric, F.Cu at (30.4, 168.4)
- added C45: 1nF, Capacitor_SMD:C_0402_1005Metric, F.Cu at (118.2, 180.4)
- added C46: 1nF, Capacitor_SMD:C_0402_1005Metric, F.Cu at (118.2, 182.4)
- added C47: 10uF, Capacitor_SMD:C_0402_1005Metric, F.Cu at (118.2, 184.3)
- added C48: 100nF, Capacitor_SMD:C_0402_1005Metric, F.Cu at (30.4, 170.4)
- added C49: .1uF, Capacitor_SMD:C_0402_1005Metric, F.Cu at (118.2, 186.3)
- added C50: 22uF, Capacitor_SMD:C_0402_1005Metric, F.Cu at (30.4, 172.3)
- added C51: 0.1uF, Capacitor_SMD:C_0402_1005Metric, F.Cu at (265.3, 21.9)
- added C52: 0.1uF, Capacitor_SMD:C_0402_1005Metric, F.Cu at (265.3, 23.9)
- added C53: 0.1uF, Capacitor_SMD:C_0402_1005Metric, F.Cu at (268.1, 20.0)
- added C54: 0.1uF, Capacitor_SMD:C_0402_1005Metric, F.Cu at (268.1, 21.9)
- added C55: 0.1uF, Capacitor_SMD:C_0402_1005Metric, F.Cu at (268.1, 23.9)
- added C56: 0.1uF, Capacitor_SMD:C_0402_1005Metric, F.Cu at (271.0, 20.0)
- added C57: 0.1uF, Capacitor_SMD:C_0402_1005Metric, F.Cu at (271.0, 21.9)
- added C58: 0.1uF, Capacitor_SMD:C_0402_1005Metric, F.Cu at (271.0, 23.9)
- added C59: 22uF, Capacitor_SMD:C_0402_1005Metric, F.Cu at (33.3, 162.5)
- added C60: 10uF, Capacitor_SMD:C_0402_1005Metric, F.Cu at (33.3, 164.5)
- added C61: 10uF, Capacitor_SMD:C_0402_1005Metric, F.Cu at (33.3, 166.4)
- added C62: 10uF, Capacitor_SMD:C_0402_1005Metric, F.Cu at (33.3, 168.4)
- added C63: 10uF, Capacitor_SMD:C_0402_1005Metric, F.Cu at (33.3, 170.4)
- added L4: 4.7uH, Inductor_SMD:L_0603_1608Metric, F.Cu at (36.7, 162.8)
- added R10: R, Resistor_SMD:R_0402_1005Metric, F.Cu at (123.1, 182.4)
- added R11: R, Resistor_SMD:R_0402_1005Metric, F.Cu at (123.1, 184.4)
- added R12: R, Resistor_SMD:R_0402_1005Metric, F.Cu at (123.1, 186.4)
- added R13: R, Resistor_SMD:R_0402_1005Metric, F.Cu at (107.6, 180.4)
- added R14: R, Resistor_SMD:R_0402_1005Metric, F.Cu at (107.6, 182.4)
- added R15: R, Resistor_SMD:R_0402_1005Metric, F.Cu at (107.6, 184.4)
- added R16: R, Resistor_SMD:R_0402_1005Metric, F.Cu at (107.6, 186.4)
- added R17: R, Resistor_SMD:R_0402_1005Metric, F.Cu at (115.4, 180.4)
- added R19: R, Resistor_SMD:R_0402_1005Metric, F.Cu at (115.4, 182.4)
- added R20: R, Resistor_SMD:R_0402_1005Metric, F.Cu at (115.4, 184.4)
- added R21: R, Resistor_SMD:R_0402_1005Metric, F.Cu at (115.4, 186.4)
- added R22: 0, Resistor_SMD:R_0402_1005Metric, F.Cu at (120.8, 177.8)
- added R28: 100R, Resistor_SMD:R_0402_1005Metric, F.Cu at (36.2, 165.0)
- added R9: R, Resistor_SMD:R_0402_1005Metric, F.Cu at (123.1, 180.4)
- C1, C10, C11, C12, C13, C14, C15, C16, C17, C18, C19, C2, C20, C21, C22, C23, C24, C25, C28, C29, C3, C30, C31, C32, C4, C5, C6, C64, C65, C66, C67, C7, C70, C71, C8, C9: footprint Capacitor_SMD:C_0603_1608Metric -> Capacitor_SMD:C_0402_1005Metric
- R1, R18, R2, R23, R24, R25, R26, R27, R29, R3, R30, R31, R32, R33, R34, R35, R36, R37, R38, R4, R40, R41, R5, R6, R7, R8: footprint Resistor_SMD:R_0603_1608Metric -> Resistor_SMD:R_0402_1005Metric
- U6: value MB85RS64V -> MB85RS64
- moved U10 144.9 mm to (44.2, 184.2)
- moved U11 144.9 mm to (44.2, 188.9)
- moved U13 144.9 mm to (49.0, 189.9)
- moved U14 144.9 mm to (49.0, 192.8)
- moved Q5 144.9 mm to (50.9, 185.2)
- moved C70 134.4 mm to (21.2, 34.2)
- moved C72 134.4 mm to (34.7, 21.6)
- moved FL1 134.4 mm to (29.0, 36.4)
- moved L3 134.4 mm to (21.2, 39.2)
- moved R26 134.4 mm to (59.9, 32.3)
- moved R39 134.4 mm to (28.7, 39.5)
- moved R41 134.4 mm to (25.2, 34.2)
- moved C27 134.4 mm to (34.7, 15.7)
- moved C28 134.4 mm to (17.2, 29.2)
- moved C29 134.4 mm to (17.2, 31.7)
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Connections:
- net /GPSRadio/RxEn Radio renamed /mcu/RxEn Radio
- net /GPSRadio/TxEN Radio renamed /mcu/TxEn Radio
- U3 pad 13: /GPSRadio/Radio/DIO1 -> /GPSRadio/Dio1 Radio
- U3 pad 14: /GPSRadio/Radio/BUSY_RF -> /GPSRadio/Busy Radio
- U3 pad 16: /GPSRadio/Radio/MISO -> /GPSRadio/Miso2
- U3 pad 17: /GPSRadio/Radio/MOSI -> /GPSRadio/Mosi2
- U3 pad 18: /GPSRadio/Radio/SCK -> /GPSRadio/Sck2
- U3 pad 19: /GPSRadio/Radio/NSS -> /GPSRadio/CS Radio
Other:
- copper layers 2 -> 4

Commit message: a
Parts:
- moved L1 54.9 mm to (140.1, 63.9)
- moved C16 54.9 mm to (136.1, 66.4)
- moved C17 54.9 mm to (136.1, 69.0)
- moved C24 49.4 mm to (119.5, 76.8)
- moved C25 49.4 mm to (119.5, 79.3)
- moved Y1 49.4 mm to (125.5, 76.7)
Changed lines of the file:
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@@
 	(footprint "VOLTV1:XTAL_ABS07-32.768KHZ-T"
 		(layer "F.Cu")
-		(at 83.36 102.49)
+		(at 125.5 76.67)
 		(property "Reference" "Y1"
 			(at -0.018 -1.8564 0)
@@
 	(footprint "Capacitor_SMD:C_0402_1005Metric"
 		(layer "F.Cu")
-		(at 77.4 102.62)
+		(at 119.54 76.8)
 		(descr "Capacitor SMD 0402 (1005 Metric), square (rectangular) end terminal, IPC-7351 nominal, (Body size source: IPC-SM-782 page 76, https://www.pcb-3d.com/wordpress/wp-content/uploads/ipc-sm-782a_amendment_1_and_2.pdf), generated with kicad-footprint-generator")
 		(tags "capacitor")
@@
 	(footprint "Capacitor_SMD:C_0402_1005Metric"
 		(layer "F.Cu")
-		(at 77.4 105.13)
+		(at 119.54 79.31)
 		(descr "Capacitor SMD 0402 (1005 Metric), square (rectangular) end terminal, IPC-7351 nominal, (Body size source: IPC-SM-782 page 76, https://www.pcb-3d.com/wordpress/wp-content/uploads/ipc-sm-782a_amendment_1_and_2.pdf), generated with kicad-footprint-generator")
 		(tags "capacitor")
@@
 	(footprint "Capacitor_SMD:C_0402_1005Metric"
 		(layer "F.Cu")
-		(at 96.3225 106.84)
+		(at 136.0725 68.95)
 		(descr "Capacitor SMD 0402 (1005 Metric), square (rectangular) end terminal, IPC-7351 nominal, (Body size source: IPC-SM-782 page 76, https://www.pcb-3d.com/wordpress/wp-content/uploads/ipc-sm-782a_amendment_1_and_2.pdf), generated with kicad-footprint-generator")
 		(tags "capacitor")
@@
 	(footprint "Capacitor_SMD:C_0402_1005Metric"
 		(layer "F.Cu")
-		(at 96.3225 104.33)
+		(at 136.0725 66.44)
 		(descr "Capacitor SMD 0402 (1005 Metric), square (rectangular) end terminal, IPC-7351 nominal, (Body size source: IPC-SM-782 page 76, https://www.pcb-3d.com/wordpress/wp-content/uploads/ipc-sm-782a_amendment_1_and_2.pdf), generated with kicad-footprint-generator")
 		(tags "capacitor")
@@
 	(footprint "Inductor_SMD:L_0603_1608Metric"
 		(layer "F.Cu")
-		(at 100.3325 101.82)
+		(at 140.0825 63.93)
 		(descr "Inductor SMD 0603 (1608 Metric), square (rectangular) end terminal, IPC-7351 nominal, (Body size source: http://www.tortai-tech.com/upload/download/2011102023233369053.pdf), generated with kicad-footprint-generator")
 		(tags "inductor")
